File: Hub1.kicad_sch (KiCad schematic)
At the start: 22 parts, among them J5 BM04B-SRSS-TB, J6 BM04B-SRSS-TB, U3 USB2422/MJ, U4 TPS2051CDBVR, U5 TPS2051CDBVR, Y2 ECS-240-8-37B-CKY-TR

Commit message: refactor: standardize project structure and link central purdue-rov-kicad-lib
Parts:
- U3: footprint ROV_PCIe_USB_HUB:QFN-24-1EP_4x4mm_P0.5mm_EP2.5x2.5mm_ThermalVias -> rov_logic:QFN-24-1EP_4x4mm_P0.5mm_EP2.5x2.5mm_ThermalVias; symbol ROV_PCIe_USB_HUB:USB2422_MJ -> rov_logic:USB2422_MJ
Changed lines of the file:
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@@
 		)
 		(instances
-			(project "ROV_PCIE_USB_HUB_FINAL"
+			(project "X19-USB-Hub-Board"
 				(path "/95e7ccb6-701a-4570-b93f-f5431fbf25de/5968cd2f-6643-449b-abda-591b3f0809fa"
 					(reference "R39")
@@
 		)
 		(instances
-			(project "ROV_PCIE_USB_HUB_FINAL"
+			(project "X19-USB-Hub-Board"
 				(path "/95e7ccb6-701a-4570-b93f-f5431fbf25de/5968cd2f-6643-449b-abda-591b3f0809fa"
 					(reference "#PWR077")
@@
 		)
 		(instances
-			(project "ROV_PCIE_USB_HUB_FINAL"
+			(project "X19-USB-Hub-Board"
 				(path "/95e7ccb6-701a-4570-b93f-f5431fbf25de/5968cd2f-6643-449b-abda-591b3f0809fa"
 					(reference "R40")
@@
 		)
 		(instances
-			(project "ROV_PCIE_USB_HUB_FINAL"
+			(project "X19-USB-Hub-Board"
 				(path "/95e7ccb6-701a-4570-b93f-f5431fbf25de/5968cd2f-6643-449b-abda-591b3f0809fa"
 					(reference "U13")
@@
 		)
 		(instances
-			(project "ROV_PCIE_USB_HUB_FINAL"
+			(project "X19-USB-Hub-Board"
 				(path "/95e7ccb6-701a-4570-b93f-f5431fbf25de/5968cd2f-6643-449b-abda-591b3f0809fa"
 					(reference "U14")
@@
 		)
 		(instances
-			(project "ROV_PCIE_USB_HUB_FINAL"
+			(project "X19-USB-Hub-Board"
 				(path "/95e7ccb6-701a-4570-b93f-f5431fbf25de/5968cd2f-6643-449b-abda-591b3f0809fa"
 					(reference "#PWR086")
@@
 		)
 		(instances
-			(project "ROV_PCIE_USB_HUB_FINAL"
+			(project "X19-USB-Hub-Board"
 				(path "/95e7ccb6-701a-4570-b93f-f5431fbf25de/5968cd2f-6643-449b-abda-591b3f0809fa"
 					(reference "#PWR084")
@@
 		)
 		(instances
-			(project "ROV_PCIE_USB_HUB_FINAL"
+			(project "X19-USB-Hub-Board"
 				(path "/95e7ccb6-701a-4570-b93f-f5431fbf25de/5968cd2f-6643-449b-abda-591b3f0809fa"
 					(reference "R42")
@@
 		)
 		(instances
-			(project "ROV_PCIE_USB_HUB_FINAL"
+			(project "X19-USB-Hub-Board"
 				(path "/95e7ccb6-701a-4570-b93f-f5431fbf25de/5968cd2f-6643-449b-abda-591b3f0809fa"
 					(reference "#PWR079")
@@
 		)
 		(instances
-			(project "ROV_PCIE_USB_HUB_FINAL"
+			(project "X19-USB-Hub-Board"
 				(path "/95e7ccb6-701a-4570-b93f-f5431fbf25de/5968cd2f-6643-449b-abda-591b3f0809fa"
 					(reference "#PWR072")
@@
 		)
 		(instances
-			(project "ROV_PCIE_USB_HUB_FINAL"
+			(project "X19-USB-Hub-Board"
 				(path "/95e7ccb6-701a-4570-b93f-f5431fbf25de/5968cd2f-6643-449b-abda-591b3f0809fa"
 					(reference "C58")
@@
 		)
 		(instances
-			(project "ROV_PCIE_USB_HUB_FINAL"
+			(project "X19-USB-Hub-Board"
 				(path "/95e7ccb6-701a-4570-b93f-f5431fbf25de/5968cd2f-6643-449b-abda-591b3f0809fa"
 					(reference "C64")
@@
 		)
 		(instances
-			(project "ROV_PCIE_USB_HUB_FINAL"
+			(project "X19-USB-Hub-Board"
 				(path "/95e7ccb6-701a-4570-b93f-f5431fbf25de/5968cd2f-6643-449b-abda-591b3f0809fa"
 					(reference "#PWR082")
@@
 		)
 		(instances
-			(project "ROV_PCIE_USB_HUB_FINAL"
+			(project "X19-USB-Hub-Board"
 				(path "/95e7ccb6-701a-4570-b93f-f5431fbf25de/5968cd2f-6643-449b-abda-591b3f0809fa"
 					(reference "J11")
@@
 		)
 		(instances
-			(project "ROV_PCIE_USB_HUB_FINAL"
+			(project "X19-USB-Hub-Board"
 				(path "/95e7ccb6-701a-4570-b93f-f5431fbf25de/5968cd2f-6643-449b-abda-591b3f0809fa"
 					(reference "#PWR085")
@@
 		)
 		(instances
-			(project "ROV_PCIE_USB_HUB_FINAL"
+			(project "X19-USB-Hub-Board"
 				(path "/95e7ccb6-701a-4570-b93f-f5431fbf25de/5968cd2f-6643-449b-abda-591b3f0809fa"
 					(reference "R41")
@@
 		)
 		(instances
-			(project "ROV_PCIE_USB_HUB_FINAL"
+			(project "X19-USB-Hub-Board"
 				(path "/95e7ccb6-701a-4570-b93f-f5431fbf25de/5968cd2f-6643-449b-abda-591b3f0809fa"
 					(reference "C56")
@@
 		)
 		(instances
-			(project "ROV_PCIE_USB_HUB_FINAL"
+			(project "X19-USB-Hub-Board"
 				(path "/95e7ccb6-701a-4570-b93f-f5431fbf25de/5968cd2f-6643-449b-abda-591b3f0809fa"
 					(reference "C61")
@@
 		)
 		(instances
-			(project "ROV_PCIE_USB_HUB_FINAL"
+			(project "X19-USB-Hub-Board"
 				(path "/95e7ccb6-701a-4570-b93f-f5431fbf25de/5968cd2f-6643-449b-abda-591b3f0809fa"
 					(reference "#PWR080")
@@
 		)
 		(instances
-			(project "ROV_PCIE_USB_HUB_FINAL"
+			(project "X19-USB-Hub-Board"
 				(path "/95e7ccb6-701a-4570-b93f-f5431fbf25de/5968cd2f-6643-449b-abda-591b3f0809fa"
 					(reference "#PWR078")
@@
 		)
 		(instances
-			(project "ROV_PCIE_USB_HUB_FINAL"
+			(project "X19-USB-Hub-Board"
 				(path "/95e7ccb6-701a-4570-b93f-f5431fbf25de/5968cd2f-6643-449b-abda-591b3f0809fa"
 					(reference "C62")
@@
 		)
 		(instances
-			(project "ROV_PCIE_USB_HUB_FINAL"
+			(project "X19-USB-Hub-Board"
 				(path "/95e7ccb6-701a-4570-b93f-f5431fbf25de/5968cd2f-6643-449b-abda-591b3f0809fa"
 					(reference "#PWR081")
@@
 		)
 		(instances
-			(project "ROV_PCIE_USB_HUB_FINAL"
+			(project "X19-USB-Hub-Board"
 				(path "/95e7ccb6-701a-4570-b93f-f5431fbf25de/5968cd2f-6643-449b-abda-591b3f0809fa"
 					(reference "R43")
@@
 		)
 		(instances
-			(project "ROV_PCIE_USB_HUB_FINAL"
+			(project "X19-USB-Hub-Board"
 				(path "/95e7ccb6-701a-4570-b93f-f5431fbf25de/5968cd2f-6643-449b-abda-591b3f0809fa"
 					(reference "C59")
@@
 		)
 		(instances
-			(project "ROV_PCIE_USB_HUB_FINAL"
+			(project "X19-USB-Hub-Board"
 				(path "/95e7ccb6-701a-4570-b93f-f5431fbf25de/5968cd2f-6643-449b-abda-591b3f0809fa"
 					(reference "C57")
@@
 		)
 		(instances
-			(project "ROV_PCIE_USB_HUB_FINAL"
+			(project "X19-USB-Hub-Board"
 				(path "/95e7ccb6-701a-4570-b93f-f5431fbf25de/5968cd2f-6643-449b-abda-591b3f0809fa"
 					(reference "Y5")
@@
 		)
 		(instances
-			(project "ROV_PCIE_USB_HUB_FINAL"
+			(project "X19-USB-Hub-Board"
 				(path "/95e7ccb6-701a-4570-b93f-f5431fbf25de/5968cd2f-6643-449b-abda-591b3f0809fa"
 					(reference "#PWR075")
@@
 	)
 	(symbol
-		(lib_id "ROV_PCIe_USB_HUB:USB2422_MJ")
+		(lib_id "rov_logic:USB2422_MJ")
 		(at 78.74 73.66 0)
 		(unit 1)
@@
 			)
 		)
-		(property "Footprint" "ROV_PCIe_USB_HUB:QFN-24-1EP_4x4mm_P0.5mm_EP2.5x2.5mm_ThermalVias"
+		(property "Footprint" "rov_logic:QFN-24-1EP_4x4mm_P0.5mm_EP2.5x2.5mm_ThermalVias"
 			(at 89.408 129.032 0)
 			(hide yes)
@@
 		)
 		(instances
-			(project "ROV_PCIE_USB_HUB_FINAL"
+			(project "X19-USB-Hub-Board"
 				(path "/95e7ccb6-701a-4570-b93f-f5431fbf25de/5968cd2f-6643-449b-abda-591b3f0809fa"
 					(reference "U12")
@@
 		)
 		(instances
-			(project "ROV_PCIE_USB_HUB_FINAL"
+			(project "X19-USB-Hub-Board"
 				(path "/95e7ccb6-701a-4570-b93f-f5431fbf25de/5968cd2f-6643-449b-abda-591b3f0809fa"
 					(reference "R38")
@@
 		)
 		(instances
-			(project "ROV_PCIE_USB_HUB_FINAL"
+			(project "X19-USB-Hub-Board"
 				(path "/95e7ccb6-701a-4570-b93f-f5431fbf25de/5968cd2f-6643-449b-abda-591b3f0809fa"
 					(reference "#PWR074")
@@
 		)
 		(instances
-			(project "ROV_PCIE_USB_HUB_FINAL"
+			(project "X19-USB-Hub-Board"
 				(path "/95e7ccb6-701a-4570-b93f-f5431fbf25de/5968cd2f-6643-449b-abda-591b3f0809fa"
 					(reference "#PWR087")
@@
 		)
 		(instances
-			(project "ROV_PCIE_USB_HUB_FINAL"
+			(project "X19-USB-Hub-Board"
 				(path "/95e7ccb6-701a-4570-b93f-f5431fbf25de/5968cd2f-6643-449b-abda-591b3f0809fa"
 					(reference "#PWR076")
@@
 		)
 		(instances
-			(project "ROV_PCIE_USB_HUB_FINAL"
+			(project "X19-USB-Hub-Board"
 				(path "/95e7ccb6-701a-4570-b93f-f5431fbf25de/5968cd2f-6643-449b-abda-591b3f0809fa"
 					(reference "J12")
@@
 		)
 		(instances
-			(project "ROV_PCIE_USB_HUB_FINAL"
+			(project "X19-USB-Hub-Board"
 				(path "/95e7ccb6-701a-4570-b93f-f5431fbf25de/5968cd2f-6643-449b-abda-591b3f0809fa"
 					(reference "C63")
@@
 		)
 		(instances
-			(project "ROV_PCIE_USB_HUB_FINAL"
+			(project "X19-USB-Hub-Board"
 				(path "/95e7ccb6-701a-4570-b93f-f5431fbf25de/5968cd2f-6643-449b-abda-591b3f0809fa"
 					(reference "C65")
@@
 		)
 		(instances
-			(project "ROV_PCIE_USB_HUB_FINAL"
+			(project "X19-USB-Hub-Board"
 				(path "/95e7ccb6-701a-4570-b93f-f5431fbf25de/5968cd2f-6643-449b-abda-591b3f0809fa"
 					(reference "#PWR073")
@@
 		)
 		(instances
-			(project "ROV_PCIE_USB_HUB_FINAL"
+			(project "X19-USB-Hub-Board"
 				(path "/95e7ccb6-701a-4570-b93f-f5431fbf25de/5968cd2f-6643-449b-abda-591b3f0809fa"
 					(reference "#PWR083")
@@
 		)
 		(instances
-			(project "ROV_PCIE_USB_HUB_FINAL"
+			(project "X19-USB-Hub-Board"
 				(path "/95e7ccb6-701a-4570-b93f-f5431fbf25de/5968cd2f-6643-449b-abda-591b3f0809fa"
 					(reference "C60")

Commit message: changes
Connections:
- net CAN+ is gone; now on net USB1_DN: J5.2 (Pin_2)
- net CAN- is gone; now on net USB1_DP: J5.3 (Pin_3)
Changed lines of the file:
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@@
+	(wire
+		(pts
+			(xy 236.22 77.47) (xy 200.66 77.47)
+		)
+		(stroke
+			(width 0)
+			(type default)
+		)
+	)
+	(wire
+		(pts
+			(xy 124.46 97.79) (xy 152.4 97.79)
+		)
+		(stroke
+			(width 0)
+			(type default)
+		)
+	)
+	(wire
+		(pts
+			(xy 55.88 114.3) (xy 58.42 114.3)
+		)
+		(stroke
+			(width 0)
+			(type default)
+		)
+	)
+	(wire
+		(pts
+			(xy 50.8 106.68) (xy 50.8 110.49)
+		)
+		(stroke
+			(width 0)
+			(type default)
+		)
+	)
+	(wire
+		(pts
+			(xy 124.46 100.33) (xy 152.4 100.33)
+		)
+		(stroke
+			(width 0)
+			(type default)
+		)
+	)
+	(wire
+		(pts
+			(xy 57.15 63.5) (xy 64.77 63.5)
+		)
+		(stroke
+			(width 0)
+			(type default)
+		)
+	)
+	(wire
+		(pts
+			(xy 50.8 110.49) (xy 55.88 110.49)
+		)
+		(stroke
+			(width 0)
+			(type default)
+		)
+	)
+	(wire
+		(pts
+			(xy 97.79 54.61) (xy 97.79 55.88)
+		)
+		(stroke
+			(width 0)
+			(type default)
+		)
+	)
+	(wire
+		(pts
+			(xy 196.85 64.77) (xy 196.85 66.04)
+		)
+		(stroke
+			(width 0)
+			(type default)
+		)
+	)
+	(wire
+		(pts
+			(xy 124.46 86.36) (xy 152.4 86.36)
+		)
+		(stroke
+			(width 0)
+			(type default)
+		)
+	)
+	(wire
+		(pts
+			(xy 64.77 57.15) (xy 64.77 55.88)
+		)
+		(stroke
+			(width 0)
+			(type default)
+		)
+	)
+	(wire
+		(pts
+			(xy 69.85 63.5) (xy 74.93 63.5)
+		)
+		(stroke
+			(width 0)
+			(type default)
+		)
+	)
 	(wire
 		(pts
 			(xy 236.22 80.01) (xy 200.66 80.01)
-		)
-		(stroke
-			(width 0)
-			(type default)
-		)
-	)
-	(wire
-		(pts
-			(xy 124.46 97.79) (xy 152.4 97.79)
-		)
-		(stroke
-			(width 0)
-			(type default)
-		)
-	)
-	(wire
-		(pts
-			(xy 55.88 114.3) (xy 58.42 114.3)
-		)
-		(stroke
-			(width 0)
-			(type default)
-		)
-	)
-	(wire
-		(pts
-			(xy 50.8 106.68) (xy 50.8 110.49)
-		)
-		(stroke
-			(width 0)
-			(type default)
-		)
-	)
-	(wire
-		(pts
-			(xy 124.46 100.33) (xy 152.4 100.33)
-		)
-		(stroke
-			(width 0)
-			(type default)
-		)
-	)
-	(wire
-		(pts
-			(xy 57.15 63.5) (xy 64.77 63.5)
-		)
-		(stroke
-			(width 0)
-			(type default)
-		)
-	)
-	(wire
-		(pts
-			(xy 50.8 110.49) (xy 55.88 110.49)
-		)
-		(stroke
-			(width 0)
-			(type default)
-		)
-	)
-	(wire
-		(pts
-			(xy 97.79 54.61) (xy 97.79 55.88)
-		)
-		(stroke
-			(width 0)
-			(type default)
-		)
-	)
-	(wire
-		(pts
-			(xy 196.85 64.77) (xy 196.85 66.04)
-		)
-		(stroke
-			(width 0)
-			(type default)
-		)
-	)
-	(wire
-		(pts
-			(xy 124.46 86.36) (xy 152.4 86.36)
-		)
-		(stroke
-			(width 0)
-			(type default)
-		)
-	)
-	(wire
-		(pts
-			(xy 64.77 57.15) (xy 64.77 55.88)
-		)
-		(stroke
-			(width 0)
-			(type default)
-		)
-	)
-	(wire
-		(pts
-			(xy 69.85 63.5) (xy 74.93 63.5)
-		)
-		(stroke
-			(width 0)
-			(type default)
-		)
-	)
-	(wire
-		(pts
-			(xy 236.22 77.47) (xy 200.66 77.47)
 		)
 		(stroke
@@
 		)
 	)
-	(label "CAN+"
-		(at 200.66 77.47 0)
+	(label "USB1_DP"
+		(at 200.66 80.01 0)
 		(effects
 			(font
@@
 		)
 	)
-	(label "CAN-"
-		(at 200.66 80.01 0)
-		(effects
-			(font
+	(label "USB1_DN"
+		(at 200.66 77.47 0)
+		(effects
+			(font

Commit message: readme + board changes
Parts:
- U3: Category (none) -> Logic; DigiKey (none) -> USB2422/MJ-ND; MPN (none) -> USB2422/MJ; Manufacturer (none) -> Microchip Technology; Temp_Range (none) -> 0°C to 70°C; Verified (none) -> Yes
Changed lines of the file:
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@@
 			)
 		)
-		(property "Datasheet" "USB2422/MJ"
+		(property "Datasheet" "https://ww1.microchip.com/downloads/en/DeviceDoc/00000062A.pdf"
 			(at 88.646 131.572 0)
 			(hide yes)
@@
 			)
 		)
-		(property "Description" ""
+		(property "Description" "2-Port USB 2.0 Hi-Speed Hub Controller, 24-QFN"
 			(at 78.74 73.66 0)
 			(hide yes)
@@
 			(at 78.74 73.66 0)
 			(hide yes)
+			(show_name no)
+			(do_not_autoplace no)
+			(effects
+				(font
+					(size 1.27 1.27)
+				)
+			)
+		)
+		(property "Manufacturer" "Microchip Technology"
+			(at 78.74 73.66 0)
+			(hide yes)
+			(show_name no)
+			(do_not_autoplace no)
+			(effects
+				(font
+					(size 1.27 1.27)
+				)
+			)
+		)
+		(property "MPN" "USB2422/MJ"
+			(at 78.74 73.66 0)
+			(hide yes)
+			(show_name no)
+			(do_not_autoplace no)
+			(effects
+				(font
+					(size 1.27 1.27)
+				)
+			)
+		)
+		(property "DigiKey" "USB2422/MJ-ND"
+			(at 78.74 73.66 0)
+			(hide yes)
+			(show_name no)
+			(do_not_autoplace no)
+			(effects
+				(font
+					(size 1.27 1.27)
+				)
+			)
+		)
+		(property "Temp_Range" "0°C to 70°C"
+			(at 78.74 73.66 0)
+			(hide yes)
+			(show_name no)
+			(do_not_autoplace no)
+			(effects
+				(font
+					(size 1.27 1.27)
+				)
+			)
+		)
+		(property "Category" "Logic"
+			(at 78.74 73.66 0)
+			(hide yes)
+			(show_name no)
+			(do_not_autoplace no)
+			(effects
+				(font
+					(size 1.27 1.27)
+				)
+			)
+		)
+		(property "Verified" "Yes"
+			(at 78.74 73.66 0)
+			(hide yes)
