File: Power.kicad_sch (KiCad schematic)
At the start: 18 parts, among them U15 TPS62A02APDDC, U16 TPS62A02APDDC

Commit message: readme + board changes
Changed lines of the file:
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@@
-		)
-	)
-	(label "3V3_EN"
-		(at 69.85 62.23 0)
-		(effects
-			(font
-				(size 1.27 1.27)
-			)
-			(justify left bottom)
-		)
-	)
-	(label "1V05_EN"
-		(at 68.58 114.3 0)
-		(effects
-			(font
-				(size 1.27 1.27)
-			)
-			(justify left bottom)
 		)
 	)
