File: X19-USB-Hub-Board.kicad_sch (KiCad schematic)
At the start: 28 parts, among them J1 SFV16R-1STBE1HLF, J2 Raspberry_Pi_4, J3 0436500227, J4 0436450200, Q1 DMP3018SFV

Commit message: refactor: standardize project structure and link central purdue-rov-kicad-lib
Parts:
- J1: footprint ROV_PCIe_USB_HUB:AMPHENOL_SFV16R-1STBE1HLF -> rov_connectors:AMPHENOL_SFV16R-1STBE1HLF; symbol ROV_PCIe_USB_HUB:SFV16R-1STBE1HLF -> rov_connectors:SFV16R-1STBE1HLF
- J3: footprint ROV_PCIe_USB_HUB:0436500227 -> rov_connectors:0436500227
Changed lines of the file:
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@@
 		)
 		(instances
-			(project "ROV_PCIE_USB_HUB_FINAL"
+			(project "X19-USB-Hub-Board"
 				(path "/95e7ccb6-701a-4570-b93f-f5431fbf25de"
 					(reference "D2")
@@
 		)
 		(instances
-			(project "ROV_PCIE_USB_HUB_FINAL"
+			(project "X19-USB-Hub-Board"
 				(path "/95e7ccb6-701a-4570-b93f-f5431fbf25de"
 					(reference "H2")
@@
 		)
 		(instances
-			(project "ROV_PCIE_USB_HUB_FINAL"
+			(project "X19-USB-Hub-Board"
 				(path "/95e7ccb6-701a-4570-b93f-f5431fbf25de"
 					(reference "#PWR010")
@@
 		)
 		(instances
-			(project "ROV_PCIE_USB_HUB_FINAL"
+			(project "X19-USB-Hub-Board"
 				(path "/95e7ccb6-701a-4570-b93f-f5431fbf25de"
 					(reference "R2")
@@
 		)
 		(instances
-			(project "ROV_PCIE_USB_HUB_FINAL"
+			(project "X19-USB-Hub-Board"
 				(path "/95e7ccb6-701a-4570-b93f-f5431fbf25de"
 					(reference "D7")
@@
 		)
 		(instances
-			(project "ROV_PCIE_USB_HUB_FINAL"
+			(project "X19-USB-Hub-Board"
 				(path "/95e7ccb6-701a-4570-b93f-f5431fbf25de"
 					(reference "H1")
@@
 		)
 		(instances
-			(project "ROV_PCIE_USB_HUB_FINAL"
+			(project "X19-USB-Hub-Board"
 				(path "/95e7ccb6-701a-4570-b93f-f5431fbf25de"
 					(reference "R5")
@@
 		)
 		(instances
-			(project "ROV_PCIE_USB_HUB_FINAL"
+			(project "X19-USB-Hub-Board"
 				(path "/95e7ccb6-701a-4570-b93f-f5431fbf25de"
 					(reference "#PWR02")
@@
 		)
 		(instances
-			(project "ROV_PCIE_USB_HUB_FINAL"
+			(project "X19-USB-Hub-Board"
 				(path "/95e7ccb6-701a-4570-b93f-f5431fbf25de"
 					(reference "#FLG02")
@@
 		)
 		(instances
-			(project "ROV_PCIE_USB_HUB_FINAL"
+			(project "X19-USB-Hub-Board"
 				(path "/95e7ccb6-701a-4570-b93f-f5431fbf25de"
 					(reference "C1")
@@
 		)
 		(instances
-			(project "ROV_PCIE_USB_HUB_FINAL"
+			(project "X19-USB-Hub-Board"
 				(path "/95e7ccb6-701a-4570-b93f-f5431fbf25de"
 					(reference "R4")
@@
 		)
 		(instances
-			(project "ROV_PCIE_USB_HUB_FINAL"
+			(project "X19-USB-Hub-Board"
 				(path "/95e7ccb6-701a-4570-b93f-f5431fbf25de"
 					(reference "J2")
@@
 		)
 		(instances
-			(project "ROV_PCIE_USB_HUB_FINAL"
+			(project "X19-USB-Hub-Board"
 				(path "/95e7ccb6-701a-4570-b93f-f5431fbf25de"
 					(reference "#PWR08")
@@
 		)
 		(instances
-			(project "ROV_PCIE_USB_HUB_FINAL"
+			(project "X19-USB-Hub-Board"
 				(path "/95e7ccb6-701a-4570-b93f-f5431fbf25de"
 					(reference "D7")
@@
 		)
 		(instances
-			(project "ROV_PCIE_USB_HUB_FINAL"
+			(project "X19-USB-Hub-Board"
 				(path "/95e7ccb6-701a-4570-b93f-f5431fbf25de"
 					(reference "#PWR05")
@@
 		)
 		(instances
-			(project "ROV_PCIE_USB_HUB_FINAL"
+			(project "X19-USB-Hub-Board"
 				(path "/95e7ccb6-701a-4570-b93f-f5431fbf25de"
 					(reference "R3")
@@
 		)
 		(instances
-			(project "ROV_PCIE_USB_HUB_FINAL"
+			(project "X19-USB-Hub-Board"
 				(path "/95e7ccb6-701a-4570-b93f-f5431fbf25de"
 					(reference "D4")
@@
 		)
 		(instances
-			(project "ROV_PCIE_USB_HUB_FINAL"
+			(project "X19-USB-Hub-Board"
 				(path "/95e7ccb6-701a-4570-b93f-f5431fbf25de"
 					(reference "D5")
@@
 		)
 		(instances
-			(project "ROV_PCIE_USB_HUB_FINAL"
+			(project "X19-USB-Hub-Board"
 				(path "/95e7ccb6-701a-4570-b93f-f5431fbf25de"
 					(reference "D3")
@@
 		)
 		(instances
-			(project "ROV_PCIE_USB_HUB_FINAL"
+			(project "X19-USB-Hub-Board"
 				(path "/95e7ccb6-701a-4570-b93f-f5431fbf25de"
 					(reference "#PWR04")
@@
 		)
 		(instances
-			(project "ROV_PCIE_USB_HUB_FINAL"
+			(project "X19-USB-Hub-Board"
 				(path "/95e7ccb6-701a-4570-b93f-f5431fbf25de"
 					(reference "D1")
@@
 		)
 		(instances
-			(project "ROV_PCIE_USB_HUB_FINAL"
+			(project "X19-USB-Hub-Board"
 				(path "/95e7ccb6-701a-4570-b93f-f5431fbf25de"
 					(reference "#FLG01")
@@
 		)
 		(instances
-			(project "ROV_PCIE_USB_HUB_FINAL"
+			(project "X19-USB-Hub-Board"
 				(path "/95e7ccb6-701a-4570-b93f-f5431fbf25de"
 					(reference "#PWR01")
@@
 		)
 		(instances
-			(project "ROV_PCIE_USB_HUB_FINAL"
+			(project "X19-USB-Hub-Board"
 				(path "/95e7ccb6-701a-4570-b93f-f5431fbf25de"
 					(reference "R8")
@@
 		)
 		(instances
-			(project "ROV_PCIE_USB_HUB_FINAL"
+			(project "X19-USB-Hub-Board"
 				(path "/95e7ccb6-701a-4570-b93f-f5431fbf25de"
 					(reference "R9")
@@
 		)
 		(instances
-			(project "ROV_PCIE_USB_HUB_FINAL"
+			(project "X19-USB-Hub-Board"
 				(path "/95e7ccb6-701a-4570-b93f-f5431fbf25de"
 					(reference "#PWR06")
@@
 		)
 		(instances
-			(project "ROV_PCIE_USB_HUB_FINAL"
+			(project "X19-USB-Hub-Board"
 				(path "/95e7ccb6-701a-4570-b93f-f5431fbf25de"
 					(reference "#PWR011")
@@
 		)
 		(instances
-			(project "ROV_PCIE_USB_HUB_FINAL"
+			(project "X19-USB-Hub-Board"
 				(path "/95e7ccb6-701a-4570-b93f-f5431fbf25de"
 					(reference "R10")
@@
 		)
 		(instances
-			(project "ROV_PCIE_USB_HUB_FINAL"
+			(project "X19-USB-Hub-Board"
 				(path "/95e7ccb6-701a-4570-b93f-f5431fbf25de"
 					(reference "D6")
@@
 		)
 		(instances
-			(project "ROV_PCIE_USB_HUB_FINAL"
+			(project "X19-USB-Hub-Board"
 				(path "/95e7ccb6-701a-4570-b93f-f5431fbf25de"
 					(reference "R7")
@@
 		)
 		(instances
-			(project "ROV_PCIE_USB_HUB_FINAL"
+			(project "X19-USB-Hub-Board"
 				(path "/95e7ccb6-701a-4570-b93f-f5431fbf25de"
 					(reference "D8")
@@
 		)
 		(instances
-			(project "ROV_PCIE_USB_HUB_FINAL"
+			(project "X19-USB-Hub-Board"
 				(path "/95e7ccb6-701a-4570-b93f-f5431fbf25de"
 					(reference "Q1")
@@
 		)
 		(instances
-			(project "ROV_PCIE_USB_HUB_FINAL"
+			(project "X19-USB-Hub-Board"
 				(path "/95e7ccb6-701a-4570-b93f-f5431fbf25de"
 					(reference "R1")
@@
 		)
 		(instances
-			(project "ROV_PCIE_USB_HUB_FINAL"
+			(project "X19-USB-Hub-Board"
 				(path "/95e7ccb6-701a-4570-b93f-f5431fbf25de"
 					(reference "H3")
@@
 			)
 		)
-		(property "Footprint" "ROV_PCIe_USB_HUB:0436500227"
+		(property "Footprint" "rov_connectors:0436500227"
 			(at 158.75 135.89 0)
 			(hide yes)
@@
 		)
 		(instances
-			(project "ROV_PCIE_USB_HUB_FINAL"
+			(project "X19-USB-Hub-Board"
 				(path "/95e7ccb6-701a-4570-b93f-f5431fbf25de"
 					(reference "J3")
@@
 	)
 	(symbol
-		(lib_id "ROV_PCIe_USB_HUB:SFV16R-1STBE1HLF")
+		(lib_id "rov_connectors:SFV16R-1STBE1HLF")
 		(at 27.94 63.5 0)
 		(unit 1)
@@
 			)
 		)
-		(property "Footprint" "ROV_PCIe_USB_HUB:AMPHENOL_SFV16R-1STBE1HLF"
+		(property "Footprint" "rov_connectors:AMPHENOL_SFV16R-1STBE1HLF"
 			(at 28.448 94.742 0)
 			(hide yes)
@@
 		)
 		(instances
-			(project "ROV_PCIE_USB_HUB_FINAL"
+			(project "X19-USB-Hub-Board"
 				(path "/95e7ccb6-701a-4570-b93f-f5431fbf25de"
 					(reference "J1")
@@
 		)
 		(instances
-			(project "ROV_PCIE_USB_HUB_FINAL"
+			(project "X19-USB-Hub-Board"
 				(path "/95e7ccb6-701a-4570-b93f-f5431fbf25de"
 					(reference "H4")
@@
 		)
 		(instances
-			(project "ROV_PCIE_USB_HUB_FINAL"
+			(project "X19-USB-Hub-Board"
 				(path "/95e7ccb6-701a-4570-b93f-f5431fbf25de"
 					(reference "#PWR07")
@@
 		)
 		(instances
-			(project "ROV_PCIE_USB_HUB_FINAL"
+			(project "X19-USB-Hub-Board"
 				(path "/95e7ccb6-701a-4570-b93f-f5431fbf25de"
 					(reference "#PWR03")
@@
 		)
 		(instances
-			(project "ROV_PCIE_USB_HUB_FINAL"
+			(project "X19-USB-Hub-Board"
 				(path "/95e7ccb6-701a-4570-b93f-f5431fbf25de"
 					(reference "R6")
@@
 		)
 		(instances
-			(project "ROV_PCIE_USB_HUB_FINAL"
+			(project "X19-USB-Hub-Board"
 				(path "/95e7ccb6-701a-4570-b93f-f5431fbf25de"
 					(reference "#PWR09")
@@
 		)
 		(instances
-			(project "ROV_PCIE_USB_HUB_FINAL"
+			(project "X19-USB-Hub-Board"
 				(path "/95e7ccb6-701a-4570-b93f-f5431fbf25de"
 					(reference "J4")
@@
 		)
 		(instances
-			(project "ROV_PCIE_USB_HUB_FINAL"
+			(project "X19-USB-Hub-Board"
 				(path "/95e7ccb6-701a-4570-b93f-f5431fbf25de"
 					(page "7")
@@
 		)
 		(instances
-			(project "ROV_PCIE_USB_HUB_FINAL"
+			(project "X19-USB-Hub-Board"
 				(path "/95e7ccb6-701a-4570-b93f-f5431fbf25de"
 					(page "6")
@@
 		)
 		(instances
-			(project "ROV_PCIE_USB_HUB_FINAL"
+			(project "X19-USB-Hub-Board"
 				(path "/95e7ccb6-701a-4570-b93f-f5431fbf25de"
 					(page "2")
@@
 		)
 		(instances
-			(project "ROV_PCIE_USB_HUB_FINAL"
+			(project "X19-USB-Hub-Board"
 				(path "/95e7ccb6-701a-4570-b93f-f5431fbf25de"
 					(page "5")
@@
 		)
 		(instances
-			(project "ROV_PCIE_USB_HUB_FINAL"
+			(project "X19-USB-Hub-Board"
 				(path "/95e7ccb6-701a-4570-b93f-f5431fbf25de"
 					(page "3")
@@
 		)
 		(instances
-			(project "ROV_PCIE_USB_HUB_FINAL"
+			(project "X19-USB-Hub-Board"
 				(path "/95e7ccb6-701a-4570-b93f-f5431fbf25de"
 					(page "4")

Commit message: readme + board changes
Parts:
- J1: Category (none) -> Connectors; DigiKey (none) -> 609-1786-1-ND; MPN (none) -> SFV16R-1STBE1HLF; Manufacturer (none) -> Amphenol ICC (FCI); Temp_Range (none) -> -55°C to 105°C; Verified (none) -> Yes
Connections:
- no-connect marks 8 -> 38
Changed lines of the file:
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@@
 	)
 	(no_connect
+		(at 27.94 161.29)
+	)
+	(no_connect
 		(at 34.29 24.13)
 	)
 	(no_connect
+		(at 93.98 148.59)
+	)
+	(no_connect
+		(at 93.98 125.73)
+	)
+	(no_connect
+		(at 93.98 158.75)
+	)
+	(no_connect
+		(at 27.94 158.75)
+	)
+	(no_connect
+		(at 27.94 151.13)
+	)
+	(no_connect
+		(at 93.98 140.97)
+	)
+	(no_connect
+		(at 27.94 148.59)
+	)
+	(no_connect
 		(at 153.67 143.51)
 	)
 	(no_connect
+		(at 27.94 168.91)
+	)
+	(no_connect
 		(at 29.21 24.13)
 	)
 	(no_connect
+		(at 93.98 163.83)
+	)
+	(no_connect
+		(at 93.98 161.29)
+	)
+	(no_connect
+		(at 93.98 133.35)
+	)
+	(no_connect
+		(at 93.98 123.19)
+	)
+	(no_connect
+		(at 27.94 125.73)
+	)
+	(no_connect
 		(at 210.82 144.78)
 	)
 	(no_connect
+		(at 27.94 140.97)
+	)
+	(no_connect
+		(at 93.98 138.43)
+	)
+	(no_connect
+		(at 93.98 156.21)
+	)
+	(no_connect
+		(at 27.94 146.05)
+	)
+	(no_connect
+		(at 93.98 166.37)
+	)
+	(no_connect
+		(at 27.94 133.35)
+	)
+	(no_connect
+		(at 93.98 146.05)
+	)
+	(no_connect
 		(at 38.1 87.63)
 	)
@@
 	)
 	(no_connect
+		(at 93.98 130.81)
+	)
+	(no_connect
+		(at 27.94 163.83)
+	)
+	(no_connect
+		(at 93.98 151.13)
+	)
+	(no_connect
+		(at 27.94 130.81)
+	)
+	(no_connect
+		(at 27.94 123.19)
+	)
+	(no_connect
+		(at 27.94 156.21)
+	)
+	(no_connect
+		(at 27.94 166.37)
+	)
+	(no_connect
+		(at 27.94 138.43)
+	)
+	(no_connect
 		(at 24.13 24.13)
 	)
@@
 		(at 39.37 24.13)
 	)
+	(no_connect
+		(at 27.94 143.51)
+	)
 	(wire
 		(pts
@@
 			)
 		)
-		(property "Datasheet" ""
+		(property "Datasheet" "https://www.amphenol-cs.com/media/wysiwyg/files/drawing/sfv_r.pdf"
 			(at 27.94 63.5 0)
 			(hide yes)
@@
 			)
 		)
-		(property "Description" ""
+		(property "Description" "FFC/FPC Connector, 0.50mm Pitch, Right-Angle, 16 Circuits, Top Contact"
 			(at 27.94 63.5 0)
 			(hide yes)
@@
 			(at 27.94 63.5 0)
 			(hide yes)
+			(show_name no)
+			(do_not_autoplace no)
+			(effects
+				(font
+					(size 1.27 1.27)
+				)
+			)
+		)
+		(property "Manufacturer" "Amphenol ICC (FCI)"
+			(at 27.94 63.5 0)
+			(hide yes)
+			(show_name no)
+			(do_not_autoplace no)
+			(effects
+				(font
+					(size 1.27 1.27)
+				)
+			)
+		)
+		(property "MPN" "SFV16R-1STBE1HLF"
+			(at 27.94 63.5 0)
+			(hide yes)
+			(show_name no)
+			(do_not_autoplace no)
+			(effects
+				(font
+					(size 1.27 1.27)
+				)
+			)
+		)
+		(property "DigiKey" "609-1786-1-ND"
+			(at 27.94 63.5 0)
+			(hide yes)
+			(show_name no)
+			(do_not_autoplace no)
+			(effects
+				(font
+					(size 1.27 1.27)
+				)
+			)
+		)
+		(property "Temp_Range" "-55°C to 105°C"
+			(at 27.94 63.5 0)
+			(hide yes)
+			(show_name no)
+			(do_not_autoplace no)
+			(effects
+				(font
+					(size 1.27 1.27)
+				)
+			)
+		)
+		(property "Category" "Connectors"
+			(at 27.94 63.5 0)
+			(hide yes)
+			(show_name no)
+			(do_not_autoplace no)
+			(effects
+				(font
+					(size 1.27 1.27)
+				)
+			)
+		)
+		(property "Verified" "Yes"
+			(at 27.94 63.5 0)
+			(hide yes)
