File: X19-USB-Hub-Board.kicad_pcb (KiCad board)
At the start: 4 copper layers, 65 x 56.5 mm, 172 parts, among them J1 SFV16R-1STBE1HLF, J10 BM04B-SRSS-TB, J11 BM04B-SRSS-TB, J12 BM04B-SRSS-TB, J2 Raspberry_Pi_4, J3 0436500227, J5 BM04B-SRSS-TB, J6 BM04B-SRSS-TB, J7 BM04B-SRSS-TB, J8 BM04B-SRSS-TB, J9 BM04B-SRSS-TB, Q1 DMP3018SFV, U1 MX25V5126FZUI, U10 TPS2051CDBV, U11 TPS2051CDBV, U12 USB2422/MJ, U13 TPS2051CDBV, U14 TPS2051CDBV, U15 TPS62A02APDDC, U16 TPS62A02APDDC, U2 UPD720201K8-7x1-BAC-A, U3 USB2422/MJ, U4 TPS2051CDBV, U5 TPS2051CDBV, U6 USB2422/MJ, U7 TPS2051CDBV, U8 TPS2051CDBV, U9 USB2422/MJ, Y1 ECS-240-8-37B-CKY-TR, Y2 ECS-240-8-37B-CKY-TR, Y3 ECS-240-8-37B-CKY-TR, Y4 ECS-240-8-37B-CKY-TR, Y5 ECS-240-8-37B-CKY-TR

Commit message: refactor: standardize project structure and link central purdue-rov-kicad-lib
Parts:
- J1: footprint ROV_PCIe_USB_HUB:AMPHENOL_SFV16R-1STBE1HLF -> rov_connectors:AMPHENOL_SFV16R-1STBE1HLF
- J3: footprint ROV_PCIe_USB_HUB:0436500227 -> rov_connectors:0436500227
- U12, U3, U6, U9: footprint ROV_PCIe_USB_HUB:QFN-24-1EP_4x4mm_P0.5mm_EP2.5x2.5mm_ThermalVias -> rov_logic:QFN-24-1EP_4x4mm_P0.5mm_EP2.5x2.5mm_ThermalVias
- U2: footprint ROV_PCIe_USB_HUB:QFN-68-1EP_8x8mm_P0.4mm_EP6.2x6.2mm -> rov_logic:QFN-68-1EP_8x8mm_P0.4mm_EP6.2x6.2mm
Changed lines of the file:
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@@
 		(property ki_fp_filters "R_*")
 		(sheetname "/")
-		(sheetfile "ROV_PCIE_USB_HUB_FINAL.kicad_sch")
+		(sheetfile "X19-USB-Hub-Board.kicad_sch")
 		(units
 			(unit
@@
 		(property ki_fp_filters "R_*")
 		(sheetname "/")
-		(sheetfile "ROV_PCIE_USB_HUB_FINAL.kicad_sch")
+		(sheetfile "X19-USB-Hub-Board.kicad_sch")
 		(units
 			(unit
@@
 		(property ki_fp_filters "MountingHole*Pad*")
 		(sheetname "/")
-		(sheetfile "ROV_PCIE_USB_HUB_FINAL.kicad_sch")
+		(sheetfile "X19-USB-Hub-Board.kicad_sch")
 		(units
 			(unit
@@
 		)
 	)
-	(footprint "ROV_PCIe_USB_HUB:QFN-24-1EP_4x4mm_P0.5mm_EP2.5x2.5mm_ThermalVias"
+	(footprint "rov_logic:QFN-24-1EP_4x4mm_P0.5mm_EP2.5x2.5mm_ThermalVias"
 		(layer "F.Cu")
 		(at 101.8 84.4 180)
@@
 		)
 	)
-	(footprint "ROV_PCIe_USB_HUB:0436500227"
+	(footprint "rov_connectors:0436500227"
 		(layer "F.Cu")
 		(at 104.299999 102.6)
@@
 		(property ki_fp_filters "TerminalBlock*:*")
 		(sheetname "/")
-		(sheetfile "ROV_PCIE_USB_HUB_FINAL.kicad_sch")
+		(sheetfile "X19-USB-Hub-Board.kicad_sch")
 		(attr through_hole)
 		(duplicate_pad_numbers_are_jumpers no)
@@
 		)
 		(embedded_fonts no)
-		(model "/Users/snadol/Desktop/ROV_PCIe_USB_HUB/lib/ROV_PCIe_USB_HUB.3d/436500227.stp"
+		(model "${KIPRJMOD}/libs/purdue-rov-kicad-lib/3D_Models/436500227.stp"
 			(offset
 				(xyz -1.5 -2 10)
@@
 		(property ki_fp_filters "R_*")
 		(sheetname "/")
-		(sheetfile "ROV_PCIE_USB_HUB_FINAL.kicad_sch")
+		(sheetfile "X19-USB-Hub-Board.kicad_sch")
 		(units
 			(unit
@@
 		(property ki_fp_filters "R_*")
 		(sheetname "/")
-		(sheetfile "ROV_PCIE_USB_HUB_FINAL.kicad_sch")
+		(sheetfile "X19-USB-Hub-Board.kicad_sch")
 		(units
 			(unit
@@
 		(property ki_fp_filters "LED* LED_SMD:* LED_THT:*")
 		(sheetname "/")
-		(sheetfile "ROV_PCIE_USB_HUB_FINAL.kicad_sch")
+		(sheetfile "X19-USB-Hub-Board.kicad_sch")
 		(units
 			(unit
@@
 		(property ki_fp_filters "LED* LED_SMD:* LED_THT:*")
 		(sheetname "/")
-		(sheetfile "ROV_PCIE_USB_HUB_FINAL.kicad_sch")
+		(sheetfile "X19-USB-Hub-Board.kicad_sch")
 		(units
 			(unit
@@
 		(property ki_fp_filters "R_*")
 		(sheetname "/")
-		(sheetfile "ROV_PCIE_USB_HUB_FINAL.kicad_sch")
+		(sheetfile "X19-USB-Hub-Board.kicad_sch")
 		(units
 			(unit
@@
 		(property ki_fp_filters "C_*")
 		(sheetname "/")
-		(sheetfile "ROV_PCIE_USB_HUB_FINAL.kicad_sch")
+		(sheetfile "X19-USB-Hub-Board.kicad_sch")
 		(units
 			(unit
@@
 		(property ki_fp_filters "MountingHole*Pad*")
 		(sheetname "/")
-		(sheetfile "ROV_PCIE_USB_HUB_FINAL.kicad_sch")
+		(sheetfile "X19-USB-Hub-Board.kicad_sch")
 		(units
 			(unit
@@
 		)
 	)
-	(footprint "ROV_PCIe_USB_HUB:QFN-68-1EP_8x8mm_P0.4mm_EP6.2x6.2mm"
+	(footprint "rov_logic:QFN-68-1EP_8x8mm_P0.4mm_EP6.2x6.2mm"
 		(layer "F.Cu")
 		(at 83.6348 74.2348 -90)
@@
 		(property ki_fp_filters "Diodes*PowerDI3333*")
 		(sheetname "/")
-		(sheetfile "ROV_PCIE_USB_HUB_FINAL.kicad_sch")
+		(sheetfile "X19-USB-Hub-Board.kicad_sch")
 		(units
 			(unit
@@
 		(property ki_fp_filters "R_*")
 		(sheetname "/")
-		(sheetfile "ROV_PCIE_USB_HUB_FINAL.kicad_sch")
+		(sheetfile "X19-USB-Hub-Board.kicad_sch")
 		(units
 			(unit
@@
 		)
 	)
-	(footprint "ROV_PCIe_USB_HUB:QFN-24-1EP_4x4mm_P0.5mm_EP2.5x2.5mm_ThermalVias"
+	(footprint "rov_logic:QFN-24-1EP_4x4mm_P0.5mm_EP2.5x2.5mm_ThermalVias"
 		(layer "F.Cu")
 		(at 63.6557 93.2041 90)
@@
 		(property ki_fp_filters "MountingHole*Pad*")
 		(sheetname "/")
-		(sheetfile "ROV_PCIE_USB_HUB_FINAL.kicad_sch")
+		(sheetfile "X19-USB-Hub-Board.kicad_sch")
 		(units
 			(unit
@@
 		(property ki_fp_filters "LED* LED_SMD:* LED_THT:*")
 		(sheetname "/")
-		(sheetfile "ROV_PCIE_USB_HUB_FINAL.kicad_sch")
+		(sheetfile "X19-USB-Hub-Board.kicad_sch")
 		(units
 			(unit
@@
 		(property ki_fp_filters "R_*")
 		(sheetname "/")
-		(sheetfile "ROV_PCIE_USB_HUB_FINAL.kicad_sch")
+		(sheetfile "X19-USB-Hub-Board.kicad_sch")
 		(units
 			(unit
@@
 		(property ki_fp_filters "LED* LED_SMD:* LED_THT:*")
 		(sheetname "/")
-		(sheetfile "ROV_PCIE_USB_HUB_FINAL.kicad_sch")
+		(sheetfile "X19-USB-Hub-Board.kicad_sch")
 		(units
 			(unit
@@
 		)
 		(sheetname "/")
-		(sheetfile "ROV_PCIE_USB_HUB_FINAL.kicad_sch")
+		(sheetfile "X19-USB-Hub-Board.kicad_sch")
 		(units
 			(unit
@@
 		(property ki_fp_filters "R_*")
 		(sheetname "/")
-		(sheetfile "ROV_PCIE_USB_HUB_FINAL.kicad_sch")
+		(sheetfile "X19-USB-Hub-Board.kicad_sch")
 		(units
 			(unit
@@
 		(property ki_fp_filters "D*SMA*")
 		(sheetname "/")
-		(sheetfile "ROV_PCIE_USB_HUB_FINAL.kicad_sch")
+		(sheetfile "X19-USB-Hub-Board.kicad_sch")
 		(units
 			(unit
@@
 		(property ki_fp_filters "R_*")
 		(sheetname "/")
-		(sheetfile "ROV_PCIE_USB_HUB_FINAL.kicad_sch")
+		(sheetfile "X19-USB-Hub-Board.kicad_sch")
 		(units
 			(unit
@@
 		)
 	)
-	(footprint "ROV_PCIe_USB_HUB:QFN-24-1EP_4x4mm_P0.5mm_EP2.5x2.5mm_ThermalVias"
+	(footprint "rov_logic:QFN-24-1EP_4x4mm_P0.5mm_EP2.5x2.5mm_ThermalVias"
 		(layer "F.Cu")
 		(at 101.8719 66.8407 180)
@@
 		(property ki_fp_filters "LED* LED_SMD:* LED_THT:*")
 		(sheetname "/")
-		(sheetfile "ROV_PCIE_USB_HUB_FINAL.kicad_sch")
+		(sheetfile "X19-USB-Hub-Board.kicad_sch")
 		(units
 			(unit
@@
 		(property ki_fp_filters "MountingHole*Pad*")
 		(sheetname "/")
-		(sheetfile "ROV_PCIE_USB_HUB_FINAL.kicad_sch")
+		(sheetfile "X19-USB-Hub-Board.kicad_sch")
 		(units
 			(unit
@@
 		(property ki_fp_filters "R_*")
 		(sheetname "/")
-		(sheetfile "ROV_PCIE_USB_HUB_FINAL.kicad_sch")
+		(sheetfile "X19-USB-Hub-Board.kicad_sch")
 		(units
 			(unit
@@
 		)
 	)
-	(footprint "ROV_PCIe_USB_HUB:QFN-24-1EP_4x4mm_P0.5mm_EP2.5x2.5mm_ThermalVias"
+	(footprint "rov_logic:QFN-24-1EP_4x4mm_P0.5mm_EP2.5x2.5mm_ThermalVias"
 		(layer "F.Cu")
 		(at 80.8 93.2 90)
@@
 		(property ki_fp_filters "SOT?323*")
 		(sheetname "/")
-		(sheetfile "ROV_PCIE_USB_HUB_FINAL.kicad_sch")
+		(sheetfile "X19-USB-Hub-Board.kicad_sch")
 		(units
 			(unit
@@
 		(embedded_fonts no)
 	)
-	(footprint "ROV_PCIe_USB_HUB:AMPHENOL_SFV16R-1STBE1HLF"
+	(footprint "rov_connectors:AMPHENOL_SFV16R-1STBE1HLF"
 		(locked yes)
 		(layer "B.Cu")
@@
 		)
 		(sheetname "/")
-		(sheetfile "ROV_PCIE_USB_HUB_FINAL.kicad_sch")
+		(sheetfile "X19-USB-Hub-Board.kicad_sch")
 		(units
 			(unit
@@
 		(property ki_fp_filters "PinHeader*2x20*P2.54mm*Vertical* PinSocket*2x20*P2.54mm*Vertical*")
 		(sheetname "/")
-		(sheetfile "ROV_PCIE_USB_HUB_FINAL.kicad_sch")
+		(sheetfile "X19-USB-Hub-Board.kicad_sch")
 		(units
 			(unit

Commit message: changes
Parts:
- U10, U11, U13, U14, U4, U5, U7, U8: value TPS2051CDBV -> TPS2051CDBVR
Changed lines of the file:
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@@
 			)
 		)
-		(property "Part Number" "RC0603FR-0710KL"
+		(property "Part Number" "RC0402FR-0710KL"
 			(at 0 0 90)
 			(unlocked yes)
@@
 			)
 		)
-		(property "Value" "TPS2051CDBV"
+		(property "Value" "TPS2051CDBVR"
 			(at 0 2.4 0)
 			(layer "F.Fab")
@@
 			)
 		)
-		(property "Part Number" "TPS2051CDBV"
+		(property "Part Number" "TPS2051CDBVR"
 			(at 0 0 180)
 			(unlocked yes)
@@
 		(sheetname "/")
 		(sheetfile "X19-USB-Hub-Board.kicad_sch")
+		(units
+			(unit
+				(name "A")
+				(pins "1" "2")
+			)
+		)
 		(attr through_hole)
 		(duplicate_pad_numbers_are_jumpers no)
@@
 			)
 		)
-		(property "Value" "TPS2051CDBV"
+		(property "Value" "TPS2051CDBVR"
 			(at 0 2.4 0)
 			(layer "F.Fab")
@@
 			)
 		)
-		(property "Part Number" "TPS2051CDBV"
+		(property "Part Number" "TPS2051CDBVR"
 			(at 0 0 180)
 			(unlocked yes)
@@
 			)
 		)
-		(property "Value" "TPS2051CDBV"
+		(property "Value" "TPS2051CDBVR"
 			(at 0 2.4 90)
 			(layer "F.Fab")
@@
 			)
 		)
-		(property "Part Number" "TPS2051CDBV"
+		(property "Part Number" "TPS2051CDBVR"
 			(at 0 0 270)
 			(unlocked yes)
@@
 			)
 		)
-		(property "Part Number" "RC0603FR-0710KL"
+		(property "Part Number" "RC0402FR-0710KL"
 			(at 0 0 0)
 			(unlocked yes)
@@
 			)
 		)
-		(property "Value" "TPS2051CDBV"
+		(property "Value" "TPS2051CDBVR"
 			(at 0 2.4 90)
 			(layer "F.Fab")
@@
 			)
 		)
-		(property "Part Number" "TPS2051CDBV"
+		(property "Part Number" "TPS2051CDBVR"
 			(at 0 0 270)
 			(unlocked yes)
@@
 			)
 		)
-		(property "Part Number" "RC0603FR-0710KL"
+		(property "Part Number" "RC0402FR-0710KL"
 			(at 0 0 90)
 			(unlocked yes)
@@
 			)
 		)
-		(property "Value" "TPS2051CDBV"
+		(property "Value" "TPS2051CDBVR"
 			(at 0 2.4 0)
 			(layer "F.Fab")
@@
 			)
 		)
-		(property "Part Number" "TPS2051CDBV"
+		(property "Part Number" "TPS2051CDBVR"
 			(at 0 0 180)
 			(unlocked yes)
@@
 			)
 		)
-		(property "Value" "TPS2051CDBV"
+		(property "Value" "TPS2051CDBVR"
 			(at 0 2.4 90)
 			(layer "F.Fab")
@@
 			)
 		)
-		(property "Part Number" "TPS2051CDBV"
+		(property "Part Number" "TPS2051CDBVR"
 			(at 0 0 270)
 			(unlocked yes)
@@
 			)
 		)
-		(property "Part Number" "RC0603FR-0710KL"
+		(property "Part Number" "RC0402FR-0710KL"
 			(at 0 0 0)
 			(unlocked yes)
@@
 			)
 		)
-		(property "Value" "TPS2051CDBV"
+		(property "Value" "TPS2051CDBVR"
 			(at 0 2.4 90)
 			(layer "F.Fab")
@@
 			)
 		)
-		(property "Part Number" "TPS2051CDBV"
+		(property "Part Number" "TPS2051CDBVR"
 			(at 0 0 270)
 			(unlocked yes)
@@
 			)
 		)
-		(property "Value" "TPS2051CDBV"
+		(property "Value" "TPS2051CDBVR"
 			(at 0 2.4 0)
 			(layer "F.Fab")
@@
 			)
 		)
-		(property "Part Number" "TPS2051CDBV"
+		(property "Part Number" "TPS2051CDBVR"
 			(at 0 0 180)
 			(unlocked yes)

Commit message: readme + board changes
Connections:
- J2 pad 1: Net-(J2-3V3-Pad1) -> unconnected-(J2-3V3-Pad1)
- J2 pad 17: Net-(J2-3V3-Pad1) -> unconnected-(J2-3V3-Pad1)_1
- J2 pad 2: Net-(J2-5V-Pad2) -> unconnected-(J2-5V-Pad2)
- J2 pad 4: Net-(J2-5V-Pad2) -> unconnected-(J2-5V-Pad2)_1
Routing:
- net Net-(J2-3V3-Pad1): track 21.4 -> 0.00 mm
- net Net-(J2-5V-Pad2): track 2.54 -> 0.00 mm
- net Net-(D6-A1): vias 4 -> 0
- removed copper zone on B.Cu, net GND
- removed copper zone on B.Cu, net Net-(D6-A1)

Commit message: updates
Parts:
- removed the G*** at (90.3, 89.4) (x2)
- added G*** (x2): LOGO, LOGO, F.Cu at (99.5, 76.4)
- added G*** (x2): LOGO, LOGO, F.Cu at (110.0, 95.9)
- added G*** (x2): LOGO, LOGO, F.Cu at (90.8, 89.6)
